Commit message: Created simple_service_server and simpler_service_client

File: src/install/bumperbot_description/share/bumperbot_description/urdf/bumperbot.urdf.xacro (robot description, xacro)
@@ -1,6 +1,11 @@
 <?xml version="1.0"?>
 <robot name="bumperbot" xmlns:xacro="http://ros.org/wiki/xacro">
+  <!--If ROS2 Humble then is_ignition = true, set to false if higher than ROS2 Humble-->
+  <!-- This is done to adapt the URDF model to the ROS2 version used-->
+  <xacro:arg name="is_ignition" default="true"/>
   <!-- Include Gazebo Parameters -->
   <xacro:include filename="$(find bumperbot_description)/urdf/bumperbot_gazebo.xacro" />
+  <!-- Include Gazebo Control Plugins (defined in the ros2 controller package) -->
+  <xacro:include filename="$(find bumperbot_description)/urdf/bumperbot_ros2_control.xacro"/>
   <link name="base_footprint"/>
   <link name="base_link">

File: src/install/bumperbot_description/share/bumperbot_description/urdf/bumperbot_gazebo.xacro (robot description, xacro)
@@ -1,4 +1,19 @@
 <?xml version = "1.0"?>
-<robot name = "bumperbot" xmlns:xacro="http://www.ros.org/wiki/xacro">
+<robot name="bumperbot" xmlns:xacro="http://www.ros.org/wiki/xacro">
+    <!-- <transmission name = "wheel_right_transmission">
+        <plugin>transmission_interface/SimpleTransmission</plugin>
+        <actuator name = "wheel_right_motor" role = "actuator_right"/>
+        <joint name = "wheel_right_joint" role = "joint_right">
+            <mechanical_reduction>1.0</mechanical_reduction>
+        </joint>
+    </transmission>
+    <transmission name = "wheel_left_transmission">
+        <plugin>transmission_interface/SimpleTransmission</plugin>
+        <actuator name = "wheel_left_motor" role = "actuator_left"/>
+        <joint name = "wheel_right_left" role = "joint_left">
+            <mechanical_reduction>1.0</mechanical_reduction>
+        </joint>
+    </transmission> -->
+    <!-- Wheels -->
     <gazebo reference = "wheel_right_link">
         <mu1>100000000000000.0</mu1>        <!-- High friction coeff to avoid slipage -->
@@ -19,4 +34,5 @@
         <fdir1>1 0 0</fdir1>                <!-- Direction of wheel rotation -->
     </gazebo>
+    <!-- Castor Wheels-->
     <gazebo reference = "castor_front_link">
         <mu1>0.1</mu1>                    <!-- High friction coeff to avoid slipage -->
@@ -35,3 +51,22 @@
         <maxVel>0.1</maxVel>
     </gazebo>
+    <gazebo>
+        <xacro:if value = "$(arg is_ignition)">
+            <plugin filename="ign_ros2_control-system" name="ign_ros2_control::IgnitionROS2ControlPlugin">
+                <parameters>$(find bumperbot_controller)/config/bumperbot_controllers.yaml</parameters>
+            </plugin>
+        </xacro:if>
+        <xacro:unless value="$(arg is_ignition)">
+            <plugin filename = "gz_ros2_control-system" name = "gz_ros2_control::GazeboSimROS2ControlPlugin">
+                <parameters>$(find bumperbot_controller)/config/bumperbot_controllers.yaml</parameters>
+            </plugin>
+        </xacro:unless>
+    </gazebo>
+    <!-- <gazebo>
+        <plugin filename = "libgazebo_ros2_control.so" name = "gazebo_ros2_control">
+            <robot_param>robot_description</robot_param>
+            <robot_param_node>robot_state_publisher</robot_param_node>
+            <parameters>$(find bumperbot_controller)/config/bumperbot_controllers.yaml</parameters>
+        </plugin>
+    </gazebo> -->
 </robot>
