Commit message: Adjust description file for control
Create new xacro file for bumperbot control, bumperbot_ros2_control.xacro, which contains the joints descriptions

Modify the xacro files in the bumperbot_description package to incorporate the necessary components for the robot control (transmission and control plugins)

File: src/bumperbot_description/urdf/bumperbot.urdf.xacro (robot description, xacro)
@@ -3,4 +3,5 @@
   <!-- Include Gazebo Parameters -->
   <xacro:include filename="$(find bumperbot_description)/urdf/bumperbot_gazebo.xacro" />
+  <xacro:include filename="$(find bumperbot_description)/urdf/bumperbot_ros2_control.xacro"/>
   <link name="base_footprint"/>
   <link name="base_link">

File: src/bumperbot_description/urdf/bumperbot_gazebo.xacro (robot description, xacro)
@@ -1,4 +1,18 @@
 <?xml version = "1.0"?>
 <robot name = "bumperbot" xmlns:xacro="http://www.ros.org/wiki/xacro">
+    <transmission name = "wheel_right_transmission">
+        <plugin>transmission_interface/SimpleTransmission</plugin>
+        <actuator name = "wheel_right_motor" role = "actuator_right"/>
+        <joint name = "wheel_right_joint" role = "joint_right">
+            <mechanical_reduction>1.0</mechanical_reduction>
+        </joint>
+    </transmission>
+    <transmission name = "wheel_left_transmission">
+        <plugin>transmission_interface/SimpleTransmission</plugin>
+        <actuator name = "wheel_left_motor" role = "actuator_left"/>
+        <joint name = "wheel_right_left" role = "joint_left">
+            <mechanical_reduction>1.0</mechanical_reduction>
+        </joint>
+    </transmission>
     <gazebo reference = "wheel_right_link">
         <mu1>100000000000000.0</mu1>        <!-- High friction coeff to avoid slipage -->
@@ -35,3 +49,10 @@
         <maxVel>0.1</maxVel>
     </gazebo>
+    <gazebo>
+        <plugin filename = "libgazebo_ros2_control.so" name = "gazebo_ros2_control">
+            <robot_param>robot_description</robot_param>
+            <robot_param_node>robot_state_pubclisherr</robot_param_node>
+            <parameters></parameters>
+        </plugin>
+    </gazebo>
 </robot>

Commit message: minor change on the material

File: src/bumperbot_description/urdf/bumperbot.urdf.xacro (robot description, xacro)
@@ -26,4 +26,12 @@
       <origin xyz="0 0 0" rpy="0 0 0" />
       <geometry>
+        <!-- Material definitions -->
+        <material name="Green">
+            <color rgba="0 0.7 0 1"/>
+        </material>
+        <material name="White">
+            <color rgba="0.7 0.7 0.7 1"/>
+        </material>
+        <!-- Base links -->
         <mesh filename="package://bumperbot_description/meshes/base_link.STL" />
       </geometry>
